File: AetherFC/SubSheet1_MCU.kicad_sch (KiCad schematic)
At the start: 23 parts, among them U3 W25Q128JVS, U6 STM32F722RETx, Y1 8MHz

Commit message: Repo cleaned up before ESC schematics
Other:
- company: (none) -> https://github.com/Lpwlk/AetherStack
