File: AetherFC/SubSheet4_Connectors.kicad_sch (KiCad schematic)
At the start: 33 parts, among them J1 SM08B, J2 SM06B, J3 SM04B, J4 USB-C socket, U7 USBLC6-2P6

Commit message: Repo cleaned up before ESC schematics
Parts:
- removed P4: ~, SolderWirePad_1x01_SMD_1x2mm, symbol MyLib:SolderPad
- added 9V, CAM, GND, RX4, TX3, TX4: ~, SolderWirePad_1x01_SMD_1x2mm, symbol MyLib:SolderPad
- renumbered P18 to 5V, P7 to 9V, P20 to BUZ+, P22 to BUZ-, P9 to CFB, P15 to GND, P19 to GND, P1 to GND, P21 to GND, P13 to M1, P12 to M2, P11 to M3, P10 to M4, P3 to RX1, P6 to RX2, P8 to RX3, P17 to RX5, SCL1 to SCL, SDA1 to SDA, P2 to TX1, P5 to TX2, P16 to TX5, P14 to Vbat
Connections:
- net 9V: now also 9V.1
- net GND: now also GND.1
- new net CAM_CTRL: CAM.1
- new net UART3_TX: TX3.1
- new net UART4_RX: RX4.1
- new net UART4_TX: TX4.1
Other:
- company: (none) -> https://github.com/Lpwlk/AetherStack
- moved on the sheet: 5V, 9V, BUZ+, BUZ-, CFB, GND, J1, J2, J3, J4, M1, M2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
